File: apic_shield_motor.sch (EAGLE design)
At the start: 9 parts, among them U1 V_REG_7805-TO220ALT, U2 V_REG_7805-TO220ALT, U3 V_REG_7805-TO220ALT, U4 V_REG_7805-TO220ALT, U5 V_REG_7805-TO220ALT, U6 V_REG_7805-TO220ALT, U7 V_REG_7805-TO220ALT, U8 V_REG_7805-TO220ALT

Commit message: update project
Parts:
- removed U1, U2, U3, U4, U5, U6, U7, U8: V_REG_7805-TO220ALT, YAEL:V_REG_7805-TO220ALT
- added C1, C2: 10uF, SparkFun-Capacitors:10UF-POLAR-RADIAL-2.5MM-25V-20%
- added D1, D2, D3, D4, D5, D6, D7, D8: 1N4004, SparkFun-DiscreteSemi:DIODE-PTH
- added J1: (no value), SparkFun-Connectors:BATTERY_CONN_DEANS
- added OK1, OK2, OK3, OK4, OK5, OK6, OK7, OK8: 4N35M, optocoupler:4N35M
- added Q1, Q2, Q3, Q4, Q5, Q6, Q7, Q8: IRF540, untitled:IRF540
- added R1, R10, R14, R17, R19, R4, R7, R9: 50k, SparkFun-Resistors:1KOHM-HORIZ-1/4W-1%
- added R11, R12, R15, R18, R2, R20, R5, R8: 1k, SparkFun-Resistors:1KOHM-HORIZ-1/4W-1%
- added R13, R16, R3, R6: 330, SparkFun-Resistors:1KOHM-HORIZ-1/4W-1%
- added X1, X2: (no value), con-ptr500:AK500/2-H
Connections:
- new net +9V: J1.+, OK1.COL, OK2.COL, OK3.COL, OK4.COL, OK5.COL, OK6.COL, OK7.COL, OK8.COL
- new net N$1: OK1.EMI, R1.2, R2.2
- new net N$10: Q3.G, R8.1
- new net N$11: Q5.G, R12.1
- new net N$12: OK6.EMI, R14.2, R15.2
- new net N$13: OK4.EMI, R10.2, R11.2
- new net N$14: Q4.G, R11.1
- new net N$15: D3.A, D4.C, Q3.S, Q4.D, X1-2.KL
- new net N$16: Q6.G, R15.1
- new net N$17: OK6.A, OK7.A, R16.1
- new net N$18: OK7.EMI, R17.2, R18.2
- new net N$19: Q7.G, R18.1
- new net N$2: Q2.G, R2.1
- new net N$20: OK8.EMI, R19.2, R20.2
- new net N$21: Q8.G, R20.1
- new net N$22: D5.A, D6.C, Q5.S, Q6.D, X2-2.KL
- new net N$23: D7.A, D8.C, Q7.S, Q8.D, X2-1.KL
- new net N$24: OK5.A, OK8.A, R13.1
- new net N$3: OK2.EMI, R4.2, R5.2
- new net N$4: OK1.A, OK4.A, R3.1
- new net N$5: Q1.G, R5.1
- new net N$6: OK5.EMI, R12.2, R9.2
- new net N$7: D1.A, D2.C, Q1.D, Q2.S, X1-1.KL
- new net N$8: OK3.EMI, R7.2, R8.2
- new net N$9: OK2.A, OK3.A, R6.1
- net +12V: now also C1.+, C2.+, D1.C, D3.C, D5.C, D7.C, J1.-, Q2.D, Q3.D, Q5.D, Q7.D
- net GND: now also C1.-, C2.-, D2.A, D4.A, D6.A, D8.A, OK1.C, OK2.C, OK3.C, OK4.C, OK5.C, OK6.C, OK7.C, OK8.C, Q1.S, Q4.S, Q6.S, Q8.S, R1.1, R10.1, R14.1, R17.1, R19.1, R4.1, R7.1, R9.1
- net RB0: now also R3.2
- net RB1: now also R6.2
- net RB2: now also R13.2
- net RB3: now also R16.2
